Commit message: adding lerobot teleop support

File: franka_emika_panda/panda.urdf (robot description, URDF)
Before this commit: robot panda, 21 links, 20 joints
Links:
- added link panda_ee
Joints:
- added joint hand_to_panda_ee_fixed: type fixed, parent hand, child panda_ee, origin xyz=0 0 0.107 rpy=0 0 0
- joint finger_joint1: axis (none) -> 0 0 1; limit (none) -> lower=0.0 upper=0.04 effort=10.0 velocity=0.1; type fixed -> prismatic
- joint finger_joint2: axis (none) -> 0 0 1; limit (none) -> lower=0.0 upper=0.04 effort=10.0 velocity=0.1; mimic (none) -> joint=finger_joint1 multiplier=1.0; type fixed -> prismatic

Commit message: Small changes

File: franka_emika_panda/panda.urdf (robot description, URDF)
Before this commit: robot panda, 22 links, 21 joints
Joints:
- joint finger_joint1: limit lower=0.0 upper=0.04 effort=10.0 velocity=0.1 -> lower=0.05 upper=0.4 effort=10.0 velocity=0.1
